File: DashRPM.kicad_sch (KiCad schematic)
At the start: 41 parts, among them J3 Conn_02x20_Odd_Even, U1 TXB0104D, U2 H11L1, U3 BTS7004-1EPP

Commit message: new file:   CLAUDE.md 	modified:   main/main.c
Parts:
- removed D1: 6A10, Diode_THT:D_P600_R-6_P20.00mm_Horizontal, symbol Diode:1N5408
- removed D10: BZT52C3V6, Diode_SMD:D_SOD-123, symbol Device:D
- removed U1: TXB0104D, Package_SO:SOIC-14_3.9x8.7mm_P1.27mm, symbol Logic_LevelTranslator:TXB0104D
- added C12, C13, C17, C18: 100nf 100v, Capacitor_SMD:C_0805_2012Metric, symbol Device:C
- added C14: 47nf 100v, Capacitor_SMD:C_0805_2012Metric, symbol Device:C
- added C15: 10nf, Capacitor_SMD:C_0805_2012Metric, symbol Device:C
- added C16: 1nf, Capacitor_SMD:C_0805_2012Metric, symbol Device:C
- added C19: 4.7nF, Capacitor_SMD:C_0805_2012Metric, symbol Device:C
- added D1, D5: BZT52C15, Diode_SMD:D_SOD-123, symbol Device:D_Zener
- added D11: 1N4148WS-HG3-08, Diode_SMD:D_SOD-323_HandSoldering, symbol Device:D
- added D6: SMBJ33A, Diode_SMD:D_SMB_Handsoldering, symbol Device:D_Zener
- added D7, D8: TBAV99,LM, Package_TO_SOT_SMD:SOT-23, symbol Diode:BAV99
- added J1: Headlight, Connector_JST:JST_XH_B2B-XH-A_1x02_P2.50mm_Vertical, symbol Connector:Conn_01x02_Pin
- added Q1: SQD50P04-09L_GE3, Package_TO_SOT_SMD:TO-252-3_TabPin2, symbol Transistor_FET:Q_PMOS_GDS
- added R14, R17: 10k, Resistor_SMD:R_1206_3216Metric_Pad1.30x1.75mm_HandSolder, symbol Device:R
- added R15, R16, R18: 4.7k, Resistor_SMD:R_0805_2012Metric_Pad1.20x1.40mm_HandSolder, symbol Device:R
- added R19, R20: 1.65k, Resistor_SMD:R_1206_3216Metric_Pad1.30x1.75mm_HandSolder, symbol Device:R
- added R21: 10k, Resistor_SMD:R_0805_2012Metric_Pad1.20x1.40mm_HandSolder, symbol Device:R
- added R22: 47k, Resistor_SMD:R_0805_2012Metric_Pad1.20x1.40mm_HandSolder, symbol Device:R
- added R23: 1k, Resistor_SMD:R_0805_2012Metric_Pad1.20x1.40mm_HandSolder, symbol Device:R
- added R3: 100k, Resistor_SMD:R_0805_2012Metric_Pad1.20x1.40mm_HandSolder, symbol Device:R
- added R4: 330, Resistor_SMD:R_0805_2012Metric_Pad1.20x1.40mm_HandSolder, symbol Device:R
- added U4, U5: SN74LVC1T45DBVR, Package_TO_SOT_SMD:SOT-23-6, symbol Logic_LevelTranslator:SN74LVC1T45DBV
- added U6: H11L1M, Package_DIP:SMDIP-6_W7.62mm, symbol Isolator:H11L1
- C1, C4, C5, C8: value 100nf -> 100nf 100v; *Mfg Part # (none) -> CL21B104KCFNNNE; LCSC (none) -> C28233; Manufacturer (none) -> Samsung Electro-Mechanics
- C10, C11, C7: value 100nf 50v -> 100nf 100v; *Mfg Part # (none) -> CL21B104KCFNNNE; LCSC (none) -> C28233; Manufacturer (none) -> Samsung Electro-Mechanics
- C2: value 1000uf 16v -> 470uf 50v; *Mfg Part # (none) -> ECA1HHG471; LCSC (none) -> C713167; Manufacturer (none) -> PANASONIC
- C3: value 100nf -> 1uF; *Mfg Part # (none) -> CL21B105KBFNNNE; LCSC (none) -> C28323; Manufacturer (none) -> Samsung Electro-Mechanics
- C6: footprint Capacitor_THT:CP_Radial_D12.5mm_P5.00mm -> Capacitor_THT:CP_Radial_D10.0mm_P5.00mm; *Mfg Part # (none) -> ECA1HHG471; LCSC (none) -> C713167; Manufacturer (none) -> PANASONIC
- C9: *Mfg Part # (none) -> CL21B222KBANNNC; LCSC (none) -> C1728; Manufacturer (none) -> Samsung Electro-Mechanics
- COIL1: value Conn_01x03_Pin -> Coil; *Mfg Part # (none) -> B3B-XH-A(LF)(SN); LCSC (none) -> C144394; Manufacturer (none) -> JST
- D2: *Mfg Part # (none) -> 5KP24CA; LCSC (none) -> C3704111; Manufacturer (none) -> Littelfuse Inc.
- D3: value SMBJ5.0A -> SMBJ6.0A; *Mfg Part # (none) -> SMBJ6.0A; LCSC (none) -> C83270; Manufacturer (none) -> Littelfuse
- D4: value SMBJ24A -> SMBJ33A; footprint Diode_SMD:D_SMB -> Diode_SMD:D_SMB_Handsoldering; *Mfg Part # (none) -> SMBJ33A; LCSC (none) -> C224019; Manufacturer (none) -> Littelfuse
- D9: value 1N4148W -> 1N4148WS-HG3-08; footprint Diode_SMD:D_SOD-123 -> Diode_SMD:D_SOD-323_HandSoldering; *Mfg Part # (none) -> 1N4148WS-HG3-08; LCSC (none) -> C3313072; Manufacturer (none) -> VISHAY
- F1: value Fuse -> 5A; *Mfg Part # (none) -> 3568; LCSC (none) -> C5249699; Manufacturer (none) -> Keystone Electronics
- F2: value Fuse -> 7.5A; *Mfg Part # (none) -> 3568; LCSC (none) -> C5249699; Manufacturer (none) -> Keystone Electronics
- J2: renamed from CarPower1; value Screw_Terminal_01x02 -> 12v In; *Mfg Part # (none) -> 1729018; LCSC (none) -> C3820334; Manufacturer (none) -> Phoenix Contact
- J3: value Conn_02x20_Odd_Even -> To Display; *Mfg Part # (none) -> 2.54-2*20P; LCSC (none) -> C9138; Manufacturer (none) -> BOOMELE(Boom Precision Elec)
- J4: renamed from AFR1; value Conn_01x04_Pin -> AFR; *Mfg Part # (none) -> B4P-VH(LF)(SN); LCSC (none) -> C160317; Manufacturer (none) -> JST
- J5: renamed from GPS1; value Conn_01x04_Pin -> GPS; *Mfg Part # (none) -> B4B-XH-A(LF)(SN); LCSC (none) -> C144395; Manufacturer (none) -> JST
- J6: renamed from 5VoltPower1; value Screw_Terminal_01x02 -> 5V In; *Mfg Part # (none) -> 1729018; LCSC (none) -> C3820334; Manufacturer (none) -> Phoenix Contact
- J7: renamed from RegulatedCarPower1; value Screw_Terminal_01x02 -> 12v out; *Mfg Part # (none) -> 1729018; LCSC (none) -> C3820334; Manufacturer (none) -> Phoenix Contact
- J8: renamed from Temp1; value Conn_01x02_Pin -> Temperature; *Mfg Part # (none) -> B2B-XH-A(LF)(SN); LCSC (none) -> C158012; Manufacturer (none) -> JST
- R1: value 1k -> 470; footprint Resistor_SMD:R_1206_3216Metric_Pad1.30x1.75mm_HandSolder -> Resistor_SMD:R_0805_2012Metric_Pad1.20x1.40mm_HandSolder; *Mfg Part # (none) -> ERJU6RD4700V; LCSC (none) -> C491182; Manufacturer (none) -> PANASONIC
- R10, R11, R12: value 1.2k -> 15k; footprint Resistor_SMD:R_1206_3216Metric_Pad1.30x1.75mm_HandSolder -> Resistor_SMD:R_2512_6332Metric_Pad1.40x3.35mm_HandSolder; *Mfg Part # (none) -> AS122WJ0153T4E; LCSC (none) -> C965951; Manufacturer (none) -> UNI-ROYAL
- R13: value 1.2k -> 2.7k; footprint Resistor_SMD:R_1206_3216Metric_Pad1.30x1.75mm_HandSolder -> Resistor_SMD:R_0805_2012Metric_Pad1.20x1.40mm_HandSolder; *Mfg Part # (none) -> ERJ6ENF2701V; LCSC (none) -> C409999; Manufacturer (none) -> PANASONIC
- R2: value 10k -> 1k; footprint Resistor_SMD:R_1206_3216Metric_Pad1.30x1.75mm_HandSolder -> Resistor_SMD:R_0805_2012Metric_Pad1.20x1.40mm_HandSolder; *Mfg Part # (none) -> ERA6AED102V; LCSC (none) -> C191555; Manufacturer (none) -> PANASONIC
- R5: value 10k -> 4.7k; footprint Resistor_SMD:R_1206_3216Metric_Pad1.30x1.75mm_HandSolder -> Resistor_SMD:R_0805_2012Metric_Pad1.20x1.40mm_HandSolder; *Mfg Part # (none) -> ERA6AEB472V; LCSC (none) -> C473295; Manufacturer (none) -> PANASONIC
- R6: footprint Resistor_SMD:R_1206_3216Metric_Pad1.30x1.75mm_HandSolder -> Resistor_SMD:R_0805_2012Metric_Pad1.20x1.40mm_HandSolder; *Mfg Part # (none) -> ERA6AEB472V; LCSC (none) -> C473295; Manufacturer (none) -> PANASONIC
- R7: value 1k -> 47; footprint Resistor_SMD:R_1206_3216Metric_Pad1.30x1.75mm_HandSolder -> Resistor_SMD:R_0805_2012Metric_Pad1.20x1.40mm_HandSolder; *Mfg Part # (none) -> ERA6VEB47R0V; LCSC (none) -> C490799; Manufacturer (none) -> PANASONIC
- R8: value 6.8k -> 8.2k; footprint Resistor_SMD:R_1206_3216Metric_Pad1.30x1.75mm_HandSolder -> Resistor_SMD:R_0805_2012Metric_Pad1.20x1.40mm_HandSolder; *Mfg Part # (none) -> ERA6AEB822V; LCSC (none) -> C445657; Manufacturer (none) -> PANASONIC
- R9: value 1k -> 4.7k; footprint Resistor_SMD:R_1206_3216Metric_Pad1.30x1.75mm_HandSolder -> Resistor_SMD:R_0805_2012Metric_Pad1.20x1.40mm_HandSolder; *Mfg Part # (none) -> ERA6AEB472V; LCSC (none) -> C473295; Manufacturer (none) -> PANASONIC
- U2: value H11L1 -> H11L1M; footprint Package_DIP:DIP-6_W7.62mm -> Package_DIP:SMDIP-6_W7.62mm; *Mfg Part # (none) -> H11L1M; LCSC (none) -> C16587; Manufacturer (none) -> onsemi
- U3: *Mfg Part # (none) -> BTS70041EPPXUMA1; LCSC (none) -> C534825; Manufacturer (none) -> Infineon Technologies
Connections:
- net 12v+: now also D1.1 (K), Q1.3 (S)
- net 3.3V+: now also C12.1, D7.2 (A), D8.2 (A), R18.1, U4.1 (VCCA), U4.5 (DIR), U5.1 (VCCA); no longer C10.2, U2.6
- net 5v+: now also C10.2, U2.6, C13.2, C18.1, R21.2, U4.6 (VCCB), U5.6 (VCCB), U6.6
- net GND: now also C11.1, J8.2 (Pin_2), C12.2, C13.1, C15.2, C16.1, C17.1, C18.2, C19.1, D11.2 (A), D5.2 (A), D6.2 (A), D7.1 (K), D8.1 (K), J1.2 (Pin_2), R14.1, R17.2, R22.2, R23.1, R3.2, U4.2 (GND), U5.2 (GND), U5.5 (DIR), U6.2, U6.5; no longer C11.2, COIL1.2 (Pin_2), R2.1
- net at C9.1, D9.1 (K), R13.2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: now also R23.2
- net at J3.37 (47), R5.2, U2.4: now also C19.2
- net at D4.1 (K), J4.1 (Pin_1), U3.10 (OUT)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: now also C15.1, R22.1
- net at C8.2, F1.2, U3.15 (VS): now also C14.1
- net at J8.1 (Pin_1), R1.1: now also C16.2, R15.1; no longer C3.2, J3.29 (51)
- net at R6.1: now also J3.29 (51), R14.2; no longer J3.18 (4)
- net at R6.2, U3.2 (IN): no longer U3.3 (DEN)
- net at D2.2 (A2), F2.2: now also Q1.2 (D)
- net at R7.2, U3.1 (GND): now also C14.2
- net at J3.11 (21): now also C11.2, R9.2, D8.3 (K); no longer J5.2 (Pin_2)
- net at J3.13 (20): now also C3.2, D7.3 (K), R15.2; no longer J5.3 (Pin_3)
- net AFR_TX: now reaches R2.2
- net AFR_TX: now also J4.2 (Pin_2); no longer J3.15 (28)
- net at J3.23 (50): now also C17.2, R18.2, U6.4
- net at J3.33 (48): now also U5.3 (A)
- net at J3.35 (52): now also U4.3 (A)
- net GPS_TX: now reaches J3.7 (29)
- net GPS_TX: now also J5.2 (Pin_2)
- net at R12.2, R13.1: now also D5.1 (K)
- net AFR_RX: now reaches J4.3 (Pin_3)
- net AFR_RX: now also R4.2
- new net: D11.1 (K), R19.2, U6.1
- new net: J3.26 (49), R16.1, R17.1
- new net: D1.2 (A), Q1.1 (G), R3.1
- new net: D6.1 (K), J1.1 (Pin_1), R20.1
- new net: R19.1, R20.2
- new net: R16.2, U3.3 (DEN)
- new net: R21.1, R4.1, U5.4 (B)
- new net: R2.1, U4.4 (B)
- new net GPS_RX: J3.15 (28), J5.3 (Pin_3)
- no-connect marks 24 -> 19
Other:
- title: (none) -> Morris Minor Dash Display
- moved on the sheet: C11, C4, C5, C6, C7, C9, COIL1, D2, D9, J8, R10, R11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
